File: PERRI_hat/PERRI_hat.kicad_pcb (KiCad board)
At the start: 2 copper layers, 163 x 100 mm, 53 parts, among them J1 ST5-80-1.00-L-D-P-TR, J2 ST5-80-1.00-L-D-P-TR, Q1 MMBT3906

Commit message: Add files via upload
Parts:
- added H1: MountingHole, PERRI_hat_footprints:Mounting_Hole_for_PERRI, F.Cu at (120.4, 130.6)
- added H2: MountingHole, PERRI_hat_footprints:Mounting_Hole_for_PERRI, F.Cu at (120.4, 48.1)
- added H3: MountingHole, PERRI_hat_footprints:Mounting_Hole_for_PERRI, F.Cu at (112.4, 130.6)
- added H4: MountingHole, PERRI_hat_footprints:Mounting_Hole_for_PERRI, F.Cu at (169.8, 48.1)
- added H5: MountingHole, PERRI_hat_footprints:Mounting_Hole_for_PERRI, F.Cu at (169.8, 130.6)
- added H6: MountingHole, PERRI_hat_footprints:Mounting_Hole_for_PERRI, F.Cu at (161.8, 130.6)
- added H7: MountingHole, PERRI_hat_footprints:Mounting_Hole_for_PERRI, F.Cu at (161.8, 48.1)
- added H8: MountingHole, PERRI_hat_footprints:Mounting_Hole_for_PERRI, F.Cu at (112.4, 48.1)
- Q1: value MMBT3906 -> MMST3904-7-F; footprint Package_TO_SOT_SMD:SOT-23 -> PERRI_hat_footprints:MMST3904-7-F
- moved R1 53.5 mm to (234.7, 41.6)
- moved R11 53.5 mm to (234.7, 58.1)
- moved R12 53.5 mm to (240.7, 58.1)
- moved R13 53.5 mm to (247.2, 58.1)
- moved R14 53.5 mm to (253.7, 58.1)
- moved R16 53.5 mm to (234.7, 66.2)
- moved R17 53.5 mm to (240.7, 66.2)
- moved R18 53.5 mm to (247.2, 66.2)
- moved R19 53.5 mm to (253.7, 66.2)
- moved R2 53.5 mm to (241.2, 41.6)
- moved R21 53.5 mm to (234.6, 74.2)
- moved R22 53.5 mm to (240.7, 74.2)
- moved R23 53.5 mm to (247.2, 74.2)
- moved R24 53.5 mm to (253.7, 74.2)
- moved R26 53.5 mm to (234.6, 81.2)
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Routing:
- net GND: track 174.1 -> 91.9 mm
- net /12V_FROM_SURF: track 35.6 -> 27.1 mm
- net /DXN: track 8.88 -> 13.9 mm
- net /DXP: track 6.66 -> 10.9 mm

Commit message: Add files via upload
Parts:
- added ?: , , F.Cu at (141.0, 103.0)
- added ?: , , F.Cu at (147.5, 79.9)
- added ?: , , F.Cu at (153.5, 72.5)
- added ?: , , F.Cu at (128.0, 94.9)
- added ?: , , F.Cu at (147.5, 94.9)
- added ?: , , F.Cu at (141.5, 65.5)
- added ?: , , F.Cu at (153.5, 110.8)
- added ?: , , F.Cu at (147.5, 86.8)
- added ?: , , F.Cu at (128.0, 72.5)
- added ?: , , F.Cu at (141.0, 79.9)
- added ?: , , F.Cu at (141.1, 94.9)
- added ?: , , F.Cu at (128.0, 65.5)
- added ?: , , F.Cu at (134.5, 79.9)
- added ?: , , F.Cu at (147.5, 110.9)
- added ?: , , F.Cu at (128.0, 80.0)
- added ?: , , F.Cu at (153.5, 103.0)
- added ?: , , F.Cu at (128.0, 86.9)
- added ?: , , F.Cu at (141.1, 86.9)
- added ?: , , F.Cu at (128.0, 110.8)
- added ?: , , F.Cu at (153.5, 52.4)
- added ?: , , F.Cu at (147.5, 102.9)
- added ?: , , F.Cu at (153.6, 94.9)
- added ?: , , F.Cu at (147.5, 58.9)
- added ?: , , F.Cu at (128.1, 58.9)
- added ?: , , F.Cu at (134.5, 58.9)
- added ?: , , F.Cu at (134.5, 94.8)
- added ?: , , F.Cu at (147.5, 72.5)
- added ?: , , F.Cu at (141.5, 72.4)
- added ?: , , F.Cu at (153.6, 86.9)
- added ?: , , F.Cu at (134.6, 65.5)
- added ?: , , F.Cu at (141.1, 110.9)
- added ?: , , F.Cu at (153.6, 59.0)
- added ?: , , F.Cu at (128.0, 102.9)
- added ?: , , F.Cu at (153.5, 65.4)
- added ?: , , F.Cu at (141.5, 59.0)
- added ?: , , F.Cu at (140.5, 119.4)
- added ?: , , F.Cu at (147.5, 65.4)
- added ?: , , F.Cu at (147.0, 119.3)
- added ?: , , F.Cu at (147.5, 52.3)
- added ?: , , F.Cu at (153.6, 119.4)
- added ?: , , F.Cu at (134.6, 72.4)
- added ?: , , F.Cu at (134.5, 102.9)
- added ?: , , F.Cu at (134.5, 110.8)
- added ?: , , F.Cu at (134.5, 86.9)
- added ?: , , F.Cu at (153.6, 79.9)
- added REF**: PERRI_ThermalVia, PERRI_hat_footprints:PERRI_ThermalVia, F.Cu at (128.5, 55.6)
- added REF**: SolderMask_Pad, PERRI_hat_footprints:SolderMask_Pad, F.Cu at (115.9, 90.0)
- added REF**: PERRI_ThermalVia, PERRI_hat_footprints:PERRI_ThermalVia, F.Cu at (142.0, 55.5)
- added REF**: PERRI_ThermalVia, PERRI_hat_footprints:PERRI_ThermalVia, F.Cu at (135.0, 55.6)
- Q1: value MMST3904-7-F -> SOT-323_DIO
- moved R5 153.3 mm to (128.0, 119.4), turned to 180 degrees
- moved R10 145.4 mm to (128.0, 110.9), turned to 180 degrees
- moved R50 143.7 mm to (128.0, 52.4), turned to 180 degrees
- moved R4 142.3 mm to (134.5, 119.4), turned to 180 degrees
- moved R15 139.5 mm to (128.0, 102.9), turned to 180 degrees
- moved R45 139.0 mm to (128.0, 58.9), turned to 180 degrees
- moved R40 135.5 mm to (128.0, 65.4), turned to 180 degrees
- moved R20 135.2 mm to (128.0, 94.9), turned to 180 degrees
- moved R9 133.7 mm to (134.5, 110.9), turned to 180 degrees
- moved R35 133.1 mm to (128.0, 72.4), turned to 180 degrees
- moved R25 132.7 mm to (128.0, 86.9), turned to 180 degrees
- moved R3 132.4 mm to (140.5, 119.4), turned to 180 degrees
- moved R30 132.1 mm to (128.0, 79.9), turned to 180 degrees
- moved R49 131.7 mm to (134.5, 52.4), turned to 180 degrees
- moved R14 127.3 mm to (134.5, 102.9), turned to 180 degrees
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Connections:
- H1 pad 1: (no net) -> GND
- H2 pad 1: (no net) -> GND
- H3 pad 1: (no net) -> GND
- H4 pad 1: (no net) -> GND
- H5 pad 1: (no net) -> GND
- H6 pad 1: (no net) -> GND
- H7 pad 1: (no net) -> GND
- H8 pad 1: (no net) -> GND
- J2 pad 02: unconnected-(J2-Pad02) -> GND
- J2 pad 04: unconnected-(J2-Pad04) -> /DXP
- J2 pad 05: /DXP -> unconnected-(J2-Pad05)
- J2 pad 07: GND -> unconnected-(J2-Pad07)
Routing:
- net GND: track 91.9 -> 0.11 mm
- net /DXN: track 13.9 -> 101.7 mm
- net /12V_FROM_SURF: track 27.1 -> 73.0 mm
- net /DXP: track 10.9 -> 9.51 mm
- added copper zone on B.Cu, net GND
Other:
- board outline removed
