File: PERRI_hat/PERRI_hat_V1.kicad_pcb (KiCad board)
At the start: 2 copper layers, 62 parts, among them J1 ST5-80-1.00-L-D-P-TR, J2 ST5-80-1.00-L-D-P-TR, Q1 MMST3904-7-F

Commit message: Add files via upload
Other:
- board outline added: 65 x 90 mm
Changed lines of the file:
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@@
     )
   )
+  (gr_line (start 107.85 39.45) (end 107.85 129.45) (layer "Edge.Cuts") (width 0.2))
+  (gr_line (start 172.85 129.45) (end 172.85 39.45) (layer "Edge.Cuts") (width 0.2))
+  (gr_line (start 107.85 129.45) (end 172.85 129.45) (layer "Edge.Cuts") (width 0.2))
+  (gr_line (start 172.85 39.45) (end 107.85 39.45) (layer "Edge.Cuts") (width 0.2))
   (segment (start 164.06 65.7) (end 165.1 65.7) (width 0.25) (layer "B.Cu") (net 152))
   (segment (start 159.7 66.2) (end 159.4 65.9) (width 0.25) (layer "B.Cu") (net 152))
@@
       (pts
         (xy 175.1 41.202353)
-        (xy 175.1 41.2)
-        (xy 176.7 122.6)
+        (xy 175.131197 41.199388)
+        (xy 176.731197 122.599388)
         (xy 176.754639 122.612304)
         (xy 176.6 133.2)
@@
         (xy 165.8 65.9)
         (xy 161.6 65.9)
-        (xy 161.2 121.1)
+        (xy 161.2 120.9)
         (xy 154.3 120.9)
         (xy 154.374957 50.077542)
@@
     )
   )
+  (group "" (id b92fc721-ba84-458f-bbfa-7844f56ca727)
+    (members
+      5c3a2310-6dbd-4c8a-b213-e2c92696148f
+      73ed45f0-88e3-4d1e-b6a8-35226ab3de7e
+      94f92153-0d03-4c84-b03c-23226eb62c53
+      a04f42a4-3b5e-44bd-a247-26d8826b7795
+    )
+  )

Commit message: Add files via upload
Parts:
- H5: value MountingHole -> (none)
Changed lines of the file:
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@@
     (property "Sheetname" "")
     (attr through_hole)
-    (fp_text reference "H3" (at 0 -0.5 unlocked) (layer "F.SilkS")
+    (fp_text reference "H3" (at 3.065 -2.58 unlocked) (layer "F.SilkS")
       (effects (font (size 1 1) (thickness 0.15)))
     )
-    (fp_text value "MountingHole" (at 0 1 unlocked) (layer "F.Fab")
-      (effects (font (size 1 1) (thickness 0.15)))
-    )
-    (fp_text user "${REFERENCE}" (at 0 2.5 unlocked) (layer "F.Fab")
+    (fp_text value "MountingHole" (at 0 1 unlocked) (layer "F.Fab") hide
       (effects (font (size 1 1) (thickness 0.15)))
     )
@@
     (property "Sheetname" "")
     (attr through_hole)
-    (fp_text reference "H2" (at 0 -0.5 unlocked) (layer "F.SilkS")
+    (fp_text reference "H2" (at 3.045 -7.23 unlocked) (layer "F.SilkS")
       (effects (font (size 1 1) (thickness 0.15)))
     )
-    (fp_text value "MountingHole" (at 0 1 unlocked) (layer "F.Fab")
-      (effects (font (size 1 1) (thickness 0.15)))
-    )
-    (fp_text user "${REFERENCE}" (at 0 2.5 unlocked) (layer "F.Fab")
+    (fp_text value "MountingHole" (at 0 1 unlocked) (layer "F.Fab") hide
       (effects (font (size 1 1) (thickness 0.15)))
     )
@@
     (property "Sheetname" "")
     (attr through_hole)
-    (fp_text reference "H6" (at 0 -0.5 unlocked) (layer "F.SilkS")
+    (fp_text reference "H6" (at -3.855 -2.47 unlocked) (layer "F.SilkS")
       (effects (font (size 1 1) (thickness 0.15)))
     )
-    (fp_text value "MountingHole" (at 0 1 unlocked) (layer "F.Fab")
-      (effects (font (size 1 1) (thickness 0.15)))
-    )
-    (fp_text user "${REFERENCE}" (at 0 2.5 unlocked) (layer "F.Fab")
+    (fp_text value "MountingHole" (at 5.705 -9.96 unlocked) (layer "F.Fab") hide
       (effects (font (size 1 1) (thickness 0.15)))
     )
@@
     (property "Sheetname" "")
     (attr through_hole)
-    (fp_text reference "H4" (at 0 -0.5 unlocked) (layer "F.SilkS")
+    (fp_text reference "H4" (at -3.855 -7.29 unlocked) (layer "F.SilkS")
       (effects (font (size 1 1) (thickness 0.15)))
     )
-    (fp_text value "MountingHole" (at 0 1 unlocked) (layer "F.Fab")
-      (effects (font (size 1 1) (thickness 0.15)))
-    )
-    (fp_text user "${REFERENCE}" (at 0 2.5 unlocked) (layer "F.Fab")
+    (fp_text value "MountingHole" (at 0 1 unlocked) (layer "F.Fab") hide
       (effects (font (size 1 1) (thickness 0.15)))
     )
@@
     (property "Sheetname" "")
     (attr through_hole)
-    (fp_text reference "H7" (at 0 -0.5 unlocked) (layer "F.SilkS")
+    (fp_text reference "H7" (at -4.025 -7.13 unlocked) (layer "F.SilkS")
       (effects (font (size 1 1) (thickness 0.15)))
     )
-    (fp_text value "MountingHole" (at 0 1 unlocked) (layer "F.Fab")
-      (effects (font (size 1 1) (thickness 0.15)))
-    )
-    (fp_text user "${REFERENCE}" (at 0 2.5 unlocked) (layer "F.Fab")
+    (fp_text value "MountingHole" (at 0 1 unlocked) (layer "F.Fab") hide
       (effects (font (size 1 1) (thickness 0.15)))
     )
@@
     (property "Sheetname" "")
     (attr through_hole)
-    (fp_text reference "H8" (at 0 -0.5 unlocked) (layer "F.SilkS")
+    (fp_text reference "H8" (at 3.125 -7.23 unlocked) (layer "F.SilkS")
       (effects (font (size 1 1) (thickness 0.15)))
     )
-    (fp_text value "MountingHole" (at 0 1 unlocked) (layer "F.Fab")
-      (effects (font (size 1 1) (thickness 0.15)))
-    )
-    (fp_text user "${REFERENCE}" (at 0 2.5 unlocked) (layer "F.Fab")
+    (fp_text value "MountingHole" (at 0 1 unlocked) (layer "F.Fab") hide
       (effects (font (size 1 1) (thickness 0.15)))
     )
@@
     (property "Sheetname" "")
     (attr through_hole)
-    (fp_text reference "H1" (at 0 -0.5 unlocked) (layer "F.SilkS")
+    (fp_text reference "H1" (at 3.345 -2.81 unlocked) (layer "F.SilkS")
       (effects (font (size 1 1) (thickness 0.15)))
     )
-    (fp_text value "MountingHole" (at 0 1 unlocked) (layer "F.Fab")
-      (effects (font (size 1 1) (thickness 0.15)))
-    )
-    (fp_text user "${REFERENCE}" (at 0 2.5 unlocked) (layer "F.Fab")
+    (fp_text value "MountingHole" (at 0 1 unlocked) (layer "F.Fab") hide
       (effects (font (size 1 1) (thickness 0.15)))
     )
@@
     (property "Sheetname" "")
     (attr through_hole)
-    (fp_text reference "H5" (at 0 -0.5 unlocked) (layer "F.SilkS")
+    (fp_text reference "H5" (at -4.075 -2.43 unlocked) (layer "F.SilkS")
       (effects (font (size 1 1) (thickness 0.15)))
     )
-    (fp_text value "MountingHole" (at 0 1 unlocked) (layer "F.Fab")
+    (fp_text value "  " (at 0 1 unlocked) (layer "F.Fab") hide
       (effects (font (size 1 1) (thickness 0.15)))
     )
-    (fp_text user "${REFERENCE}" (at 0 2.5 unlocked) (layer "F.Fab")
-      (effects (font (size 1 1) (thickness 0.15)))
-    )

Commit message: Add files via upload
Parts:
- moved R43 6.12 mm to (140.7, 65.0)
- moved R38 6.12 mm to (140.7, 71.5)
- moved R48 6.12 mm to (140.7, 58.5)
- moved R37 6.09 mm to (147.2, 71.5)
- moved R42 6.07 mm to (147.2, 65.0)
- moved R44 6.07 mm to (134.2, 65.0)
- moved R39 6.07 mm to (134.2, 71.5)
- moved R47 6.07 mm to (147.2, 58.5)
- moved R49 6.07 mm to (134.2, 58.5)
- moved R40 6.07 mm to (127.7, 71.5)
- moved R45 6.07 mm to (127.7, 65.0)
- moved R50 6.07 mm to (127.7, 58.5)
- moved R36 6.06 mm to (153.7, 71.5)
- moved R46 6.06 mm to (153.7, 58.5)
- moved R41 6.06 mm to (153.7, 65.0)
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Routing:
- net GND: track 725.4 -> 727.6 mm
- net Net-(R6-Pad2): track 3.07 -> 3.58 mm
- net Net-(R47-Pad2): track 3.07 -> 3.58 mm
- net Net-(R46-Pad2): track 3.07 -> 3.58 mm
- net Net-(R37-Pad2): track 3.07 -> 3.58 mm
- net Net-(R36-Pad2): track 3.07 -> 3.58 mm
- net Net-(R32-Pad2): track 3.07 -> 3.58 mm
- net Net-(R31-Pad2): track 3.07 -> 3.58 mm
- net Net-(R16-Pad2): track 3.07 -> 3.58 mm
- net Net-(R11-Pad2): track 3.07 -> 3.58 mm
- net Net-(R43-Pad2): track 4.07 -> 3.57 mm
- net Net-(R42-Pad2): track 3.07 -> 3.57 mm
- net Net-(R41-Pad2): track 3.07 -> 3.57 mm
