File: PERRI_hat/PERRI_hat_V1.kicad_pcb (KiCad board)
At the start: 2 copper layers, 65 x 90 mm, 62 parts, among them J1 ST5-80-1.00-L-D-P-TR, J2 ST5-80-1.00-L-D-P-TR, Q1 MMST3904-7-F

Commit message: Add files via upload
Parts:
- H5: value (none) -> MountingHole
Connections:
- Q1 pad 3: GND -> /DXP
Routing:
- net GND: track 727.6 -> 756.7 mm
- net /DXP: track 12.9 -> 21.4 mm
- net /12V_FROM_SURF: track 3.03 -> 7.99 mm

Commit message: Add files via upload
Connections:
- J2 pad 09: unconnected-(J2-Pad09) -> /12V_FROM_SURF
Routing:
- net /12V_FROM_SURF: track 7.99 -> 13.8 mm
