File: PERRI_hat/PERRI_hat.kicad_sch (KiCad schematic)
At the start: 53 parts, among them J1 ST5-80-1.00-L-D-P-TR, J2 ST5-80-1.00-L-D-P-TR, Q1 MMBT3906

Commit message: Add files via upload
Parts:
- Q1: value MMBT3906 -> MMST3904-7-F; footprint Package_TO_SOT_SMD:SOT-23 -> PERRI_hat_footprints:MMST3904-7-F
Connections:
- net DXN: now also J2.03; no longer J2.05
- net DXP: now also J2.05; no longer J2.03
- no-connect marks 0 -> 316

Commit message: Add files via upload
Parts:
- added H1, H2, H3, H4, H5, H6, H7, H8: MountingHole, PERRI_hat_footprints:Mounting_Hole_for_PERRI, symbol Mechanical:MountingHole
Connections:
- net DXP: now also J2.04; no longer J2.05
- net GND: now also J2.10; no longer J2.07
Other:
- moved on the sheet: J2B

Commit message: Add files via upload
Connections:
- net 12V_FROM_SURF: now also J2.02, J2.03, J2.04, J2.05, J2.06, J2.07
- net DXN: now also J1.01; no longer J2.03
- net DXP: now also J1.03; no longer J2.04
- net GND: now also J1.15, J1.23, J1.31, J1.39, J1.47, J1.55, J1.63, J2.16, J2.22, J2.28, J2.34, J2.40, J2.46
- no-connect marks 316 -> 297
